File: KiCAD/PiHat/pihat/pihat.sch (KiCad schematic (older format))
At the start: 43 parts, among them J1 Pan Servo Connector, J2 Tilt Servo Connector, J3 Fan, J4 Power Connector, P1 Conn_02x20_Odd_Even, P2 Pad, P3 Pad, P4 Pad, P5 Pad, P6 Pad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

Commit message: Revision 1
Parts:
- added C6: 47 uF, Capacitor_SMD:C_1206_3216Metric_Pad1.42x1.75mm_HandSolder, symbol Device:C_Small
- added F1: 5A Medium Blow, Resistor_SMD:R_0603_1608Metric_Pad1.05x0.95mm_HandSolder, symbol Device:Fuse
- C1: value 100 uF -> 47 uF; footprint Resistor_SMD:R_1206_3216Metric -> Capacitor_SMD:C_1206_3216Metric_Pad1.42x1.75mm_HandSolder
- L1: footprint trailTracer:Coil -> trailTracer:SRR1050A Coil
Connections:
- net GND: now also C6.2
- net Pi_Power+ renamed +12V
- net +12V: now also C6.1, F1.2; no longer J4.2 (Pin_2)
- new net: F1.1, J4.2 (Pin_2)
Other:
- moved on the sheet: C1, D3, R10
Changed lines of the file:
@@
 EESchema Schematic File Version 4
-LIBS:pihat-cache
 EELAYER 30 0
 EELAYER END
@@
 F1 "Power.sch" 50
 $EndSheet
-Text GLabel 2250 9600 0    50   Input ~ 0
-Pi_Power+
 $Comp
 L Device:C_Small C1
 U 1 1 5E594CA8
-P 2600 9800
-F 0 "C1" H 2692 9846 50  0000 L CNN
-F 1 "100 uF" H 2692 9755 50  0000 L CNN
-F 2 "Resistor_SMD:R_1206_3216Metric" H 2600 9800 50  0001 C CNN
-F 3 "~" H 2600 9800 50  0001 C CNN
-	1    2600 9800
+P 2800 9800
+F 0 "C1" H 2892 9846 50  0000 L CNN
+F 1 "47 uF" H 2892 9755 50  0000 L CNN
+F 2 "Capacitor_SMD:C_1206_3216Metric_Pad1.42x1.75mm_HandSolder" H 2800 9800 50  0001 C CNN
+F 3 "~" H 2800 9800 50  0001 C CNN
+	1    2800 9800
 	1    0    0    -1
 $EndComp
@@
 L power:GND #PWR0109
 U 1 1 5E59A100
-P 2600 10000
-F 0 "#PWR0109" H 2600 9750 50  0001 C CNN
-F 1 "GND" H 2605 9827 50  0000 C CNN
-F 2 "" H 2600 10000 50  0001 C CNN
-F 3 "" H 2600 10000 50  0001 C CNN
-	1    2600 10000
-	1    0    0    -1
-$EndComp
-Wire Wire Line
-	2600 10000 2600 9900
+P 2800 10000
+F 0 "#PWR0109" H 2800 9750 50  0001 C CNN
+F 1 "GND" H 2805 9827 50  0000 C CNN
+F 2 "" H 2800 10000 50  0001 C CNN
+F 3 "" H 2800 10000 50  0001 C CNN
+	1    2800 10000
+	1    0    0    -1
+$EndComp
+Wire Wire Line
+	2800 10000 2800 9900
 $Comp
 L power:GND #PWR0110
@@
 $EndComp
 Connection ~ 9250 5000
-Text GLabel 13850 4550 2    50   Input ~ 0
-Pi_Power+
-Text GLabel 13800 4000 1    50   Input ~ 0
-Pi_Power+
-Wire Wire Line
-	13700 4250 13700 4600
 $Comp
 L power:GND #PWR0108
 U 1 1 5E4EF4E1
-P 13700 4600
-F 0 "#PWR0108" H 13700 4350 50  0001 C CNN
-F 1 "GND" H 13705 4427 50  0000 C CNN
-F 2 "" H 13700 4600 50  0001 C CNN
-F 3 "" H 13700 4600 50  0001 C CNN
-	1    13700 4600
+P 13500 4500
+F 0 "#PWR0108" H 13500 4250 50  0001 C CNN
+F 1 "GND" H 13505 4327 50  0000 C CNN
+F 2 "" H 13500 4500 50  0001 C CNN
+F 3 "" H 13500 4500 50  0001 C CNN
+	1    13500 4500
 	1    0    0    -1
 $EndComp
@@
 Wire Wire Line
 	9550 4350 9550 4100
-Wire Wire Line
-	9550 4700 9550 4550
 $Comp
 L Device:R_Small R4
@@
 L power:+3.3V #PWR0101
 U 1 1 5E50C3EE
-P 9850 4700
-F 0 "#PWR0101" H 9850 4550 50  0001 C CNN
-F 1 "+3.3V" H 9865 4873 50  0000 C CNN
-F 2 "" H 9850 4700 50  0001 C CNN
-F 3 "" H 9850 4700 50  0001 C CNN
-	1    9850 4700
+P 9850 4650
+F 0 "#PWR0101" H 9850 4500 50  0001 C CNN
+F 1 "+3.3V" H 9865 4823 50  0000 C CNN
+F 2 "" H 9850 4650 50  0001 C CNN
+F 3 "" H 9850 4650 50  0001 C CNN
+	1    9850 4650
 	-1   0    0    1
 $EndComp
-Wire Wire Line
-	9850 4700 9850 4400
-Connection ~ 9850 4400
 $Comp
 L trailTracer:TPS5430-Q1 U1
@@
 F 0 "L1" V 5440 9600 50  0000 C CNN
 F 1 "15 uH" V 5349 9600 50  0000 C CNN
-F 2 "trailTracer:Coil" H 5250 9600 50  0001 C CNN
+F 2 "trailTracer:SRR1050A Coil" H 5250 9600 50  0001 C CNN
 F 3 "~" H 5250 9600 50  0001 C CNN
 	1    5250 9600
 	0    -1   -1   0
 $EndComp
-Wire Wire Line
-	2250 9600 2600 9600
-Wire Wire Line
-	2600 9700 2600 9600
-Connection ~ 2600 9600
-Wire Wire Line
-	2600 9600 3250 9600
 Wire Wire Line
 	4300 10400 6000 10400
@@
 L power:+5V #PWR0117
 U 1 1 5E6212D3
-P 7250 7200
-F 0 "#PWR0117" H 7250 7050 50  0001 C CNN
-F 1 "+5V" H 7265 7373 50  0000 C CNN
-F 2 "" H 7250 7200 50  0001 C CNN
-F 3 "" H 7250 7200 50  0001 C CNN
-	1    7250 7200
+P 7250 7050
+F 0 "#PWR0117" H 7250 6900 50  0001 C CNN
+F 1 "+5V" H 7265 7223 50  0000 C CNN
+F 2 "" H 7250 7050 50  0001 C CNN
+F 3 "" H 7250 7050 50  0001 C CNN
+	1    7250 7050
 	1    0    0    -1
 $EndComp
 Wire Wire Line
 	7250 7750 7400 7750
-Wire Wire Line
-	7250 7200 7250 7300
 Wire Wire Line
 	7900 7350 7900 7300
@@
 	1    0    0    -1
 $EndComp
-Wire Wire Line
-	4700 1300 5000 1300
-Connection ~ 4700 1300
-Text GLabel 5000 1300 2    50   Input ~ 0
+Text GLabel 4850 1300 2    50   Input ~ 0
 PI_5V
 Wire Wire Line
@@
 L power:+5V #PWR0120
 U 1 1 5E855ABE
-P 9550 4700
-F 0 "#PWR0120" H 9550 4550 50  0001 C CNN
-F 1 "+5V" H 9565 4873 50  0000 C CNN
-F 2 "" H 9550 4700 50  0001 C CNN
-F 3 "" H 9550 4700 50  0001 C CNN
-	1    9550 4700
+P 9550 4650
+F 0 "#PWR0120" H 9550 4500 50  0001 C CNN
+F 1 "+5V" H 9565 4823 50  0000 C CNN
+F 2 "" H 9550 4650 50  0001 C CNN
+F 3 "" H 9550 4650 50  0001 C CNN
+	1    9550 4650
 	-1   0    0    1
 $EndComp
@@
 L Device:LED D3
 U 1 1 5E8748D2
-P 14750 4300
-F 0 "D3" H 14743 4045 50  0000 C CNN
-F 1 "LED" H 14743 4136 50  0000 C CNN
-F 2 "LED_THT:LED_D3.0mm" H 14750 4300 50  0001 C CNN
-F 3 "~" H 14750 4300 50  0001 C CNN
-	1    14750 4300
+P 14450 4650
+F 0 "D3" H 14443 4395 50  0000 C CNN
+F 1 "LED" H 14443 4486 50  0000 C CNN
+F 2 "LED_THT:LED_D3.0mm" H 14450 4650 50  0001 C CNN
+F 3 "~" H 14450 4650 50  0001 C CNN
+	1    14450 4650
 	-1   0    0    1
 $EndComp
-Wire Wire Line
-	13800 4550 13850 4550
 $Comp
 L power:GND #PWR0119
 U 1 1 5E88C95A
-P 15000 4400
-F 0 "#PWR0119" H 15000 4150 50  0001 C CNN
-F 1 "GND" H 15005 4227 50  0000 C CNN
-F 2 "" H 15000 4400 50  0001 C CNN
-F 3 "" H 15000 4400 50  0001 C CNN
-	1    15000 4400
-	1    0    0    -1
-$EndComp
-Wire Wire Line
-	14900 4300 15000 4300
-Wire Wire Line
-	15000 4300 15000 4400
-Wire Wire Line
-	13800 4250 13800 4300
+P 14700 4750
+F 0 "#PWR0119" H 14700 4500 50  0001 C CNN
+F 1 "GND" H 14705 4577 50  0000 C CNN
+F 2 "" H 14700 4750 50  0001 C CNN
+F 3 "" H 14700 4750 50  0001 C CNN
+	1    14700 4750
+	1    0    0    -1
+$EndComp
+Wire Wire Line
+	14600 4650 14700 4650
+Wire Wire Line
+	14700 4650 14700 4750
 $Comp
 L Device:R_Small R10
 U 1 1 5E89A304
-P 14200 4300
-F 0 "R10" V 14300 4150 50  0000 C CNN
-F 1 "470" V 14300 4400 50  0000 C CNN
-F 2 "Resistor_SMD:R_0805_2012Metric_Pad1.15x1.40mm_HandSolder" H 14200 4300 50  0001 C CNN
-F 3 "~" H 14200 4300 50  0001 C CNN
-	1    14200 4300
+P 13900 4650
+F 0 "R10" V 14000 4950 50  0000 C CNN
+F 1 "470" V 14000 4750 50  0000 C CNN
+F 2 "Resistor_SMD:R_0805_2012Metric_Pad1.15x1.40mm_HandSolder" H 13900 4650 50  0001 C CNN
+F 3 "~" H 13900 4650 50  0001 C CNN
+	1    13900 4650
 	0    1    1    0
 $EndComp
@@
 $EndComp
 Wire Wire Line
-	13800 4300 14100 4300
-Connection ~ 13800 4300
-Wire Wire Line
-	13800 4300 13800 4550
-Wire Wire Line
-	14300 4300 14600 4300
+	14000 4650 14300 4650
 $Comp
 L Device:LED D4
@@
 Wire Wire Line
 	12400 9650 12250 9650
+$Comp
+L power:+12V #PWR0123
+U 1 1 5E72375F
+P 2250 9450
+F 0 "#PWR0123" H 2250 9300 50  0001 C CNN
+F 1 "+12V" H 2265 9623 50  0000 C CNN
+F 2 "" H 2250 9450 50  0001 C CNN
+F 3 "" H 2250 9450 50  0001 C CNN
+	1    2250 9450
+	1    0    0    -1
+$EndComp
+Wire Wire Line
+	2250 9450 2250 9600
+Wire Wire Line
+	4700 1300 4850 1300
+Connection ~ 4700 1300
+Wire Wire Line
+	9850 4400 9850 4650
+Connection ~ 9850 4400
+Wire Wire Line
+	9550 4550 9550 4650
+$Comp
+L power:+12V #PWR0124
+U 1 1 5E70259E
+P 13800 4900
+F 0 "#PWR0124" H 13800 4750 50  0001 C CNN
+F 1 "+12V" H 13650 5050 50  0000 L CNN
+F 2 "" H 13800 4900 50  0001 C CNN
+F 3 "" H 13800 4900 50  0001 C CNN
+	1    13800 4900
+	-1   0    0    1
+$EndComp
+$Comp
+L Device:Fuse F1
+U 1 1 5E78D052
+P 13800 4400
+F 0 "F1" H 13860 4446 50  0000 L CNN
+F 1 "5A Medium Blow" H 13860 4355 50  0000 L CNN
+F 2 "Resistor_SMD:R_0603_1608Metric_Pad1.05x0.95mm_HandSolder" V 13730 4400 50  0001 C CNN
+F 3 "~" H 13800 4400 50  0001 C CNN
+	1    13800 4400
+	1    0    0    -1
+$EndComp
+$Comp
+L Device:C_Small C6
+U 1 1 5E7A825B
+P 2500 9800
+F 0 "C6" H 2250 9850 50  0000 L CNN
+F 1 "47 uF" H 2150 9750 50  0000 L CNN
+F 2 "Capacitor_SMD:C_1206_3216Metric_Pad1.42x1.75mm_HandSolder" H 2500 9800 50  0001 C CNN
+F 3 "~" H 2500 9800 50  0001 C CNN
+	1    2500 9800
+	1    0    0    -1
+$EndComp
+$Comp
+L power:GND #PWR0125
+U 1 1 5E7A8261
+P 2500 10000
+F 0 "#PWR0125" H 2500 9750 50  0001 C CNN
+F 1 "GND" H 2505 9827 50  0000 C CNN
+F 2 "" H 2500 10000 50  0001 C CNN
+F 3 "" H 2500 10000 50  0001 C CNN
+	1    2500 10000
+	1    0    0    -1
+$EndComp
+Wire Wire Line
+	2500 10000 2500 9900
+Wire Wire Line
+	2250 9600 2500 9600
+Wire Wire Line
+	2500 9700 2500 9600
+Connection ~ 2500 9600
+Wire Wire Line
+	2500 9600 2800 9600
+Wire Wire Line
+	2800 9600 2800 9700
+Connection ~ 2800 9600
+Wire Wire Line
+	2800 9600 3250 9600
+Wire Wire Line
+	7250 7050 7250 7300
+Wire Wire Line
+	13700 4250 13500 4250
+Wire Wire Line
+	13500 4250 13500 4500
+Wire Wire Line
+	13800 4550 13800 4650
+Wire Wire Line
+	13800 4650 13800 4900
+Connection ~ 13800 4650
 $EndSCHEMATC

Commit message: Re-routing of components, fixed bugs from first spin
Parts:
- removed C4: 10nF, Resistor_SMD:R_1206_3216Metric_Pad1.42x1.75mm_HandSolder, symbol Device:C_Small
- removed D1: B340, trailTracer:DO-214, symbol Diode:B340
- removed P2, P3, P5, P6, P7: Pad, trailTracer:Pad, symbol trailTracer:Pad
- added D5: B340, Diode_THT:D_DO-15_P5.08mm_Vertical_AnodeUp, symbol Diode:B340
- P4: symbol trailTracer:Pad -> pihat-rescue:Pad-trailTracer
- U1: symbol trailTracer:TPS5430-Q1 -> pihat-rescue:TPS5430-Q1-trailTracer
- U3: symbol trailTracer:ATTiny85 -> pihat-rescue:ATTiny85-trailTracer
- U4: symbol trailTracer:TE_OJ-SH-105LM -> pihat-rescue:TE_OJ-SH-105LM-trailTracer
Connections:
- net GND: now also D5.2 (A)
- net at C2.1, L1.1, U1.8 (PH): now also D5.1 (K)
- net at U3.1 (PB5): no longer U2.1 (Vout)
- net at R11.1, R9.1: now also U3.3 (PB4); no longer U3.2 (PB3)
- net TINY_B2: now reaches U3.7 (PB2)
- net TINY_B2: now also U2.1 (Vout)
- net TINY_B4: now reaches D2.1 (K), U4.1 (COIL_1)
- net TINY_B4: now also U3.2 (PB3)
- net GPIO14(TXD0) renamed GPIO_14
- net GPIO15(RXD0) renamed GPIO_15
Other:
- note removed: "P7: Jump to ATTiny85 output pad.\n"
- moved on the sheet: P4, R11, R9
Changed lines of the file:
@@
 $EndComp
 $Comp
-L trailTracer:TPS5430-Q1 U1
+L pihat-rescue:TPS5430-Q1-trailTracer U1
 U 1 1 5E62FD94
 P 3700 9800
@@
 Wire Wire Line
 	5400 9600 5550 9600
-Connection ~ 4950 9600
 Wire Wire Line
 	5550 9600 5550 9700
-Wire Wire Line
-	4950 9600 5100 9600
-Wire Wire Line
-	4950 9700 4950 9600
 $Comp
 L Device:CP1_Small C3
@@
 	1    5550 9800
 	1    0    0    -1
-$EndComp
-Wire Wire Line
-	4950 10000 4950 10100
-$Comp
-L power:GND #PWR0111
-U 1 1 5E5B6D0F
-P 4950 10100
-F 0 "#PWR0111" H 4950 9850 50  0001 C CNN
-F 1 "GND" H 4955 9927 50  0000 C CNN
-F 2 "" H 4950 10100 50  0001 C CNN
-F 3 "" H 4950 10100 50  0001 C CNN
-	1    4950 10100
-	1    0    0    -1
-$EndComp
-$Comp
-L Diode:B340 D1
-U 1 1 5E5B50E4
-P 4950 9850
-F 0 "D1" V 4904 9929 50  0000 L CNN
-F 1 "B340" V 4995 9929 50  0000 L CNN
-F 2 "trailTracer:DO-214" H 4950 9675 50  0001 C CNN
-F 3 "http://www.jameco.com/Jameco/Products/ProdDS/1538777.pdf" H 4950 9850 50  0001 C CNN
-	1    4950 9850
-	0    1    1    0
 $EndComp
 $Comp
@@
 Wire Wire Line
 	4150 10200 4150 10450
-Wire Wire Line
-	4650 9600 4950 9600
 Connection ~ 4650 9600
 Connection ~ 5550 9600
-Wire Wire Line
-	8600 7750 8600 8750
 Connection ~ 7250 7750
 Wire Wire Line
@@
 $EndComp
 Wire Wire Line
-	8600 8750 8800 8750
-Wire Wire Line
 	8400 7750 8600 7750
 Wire Wire Line
@@
 Connection ~ 6000 9600
 $Comp
-L trailTracer:ATTiny85 U3
+L pihat-rescue:ATTiny85-trailTracer U3
 U 1 1 5E5C840A
 P 9200 9000
@@
 	1    0    0    -1
 $EndComp
-Wire Wire Line
-	9750 8750 9600 8750
 $Comp
 L power:GND #PWR0115
@@
 Wire Wire Line
 	8800 9200 8650 9200
-Wire Wire Line
-	9750 8350 9750 8500
-Connection ~ 9750 8500
-Wire Wire Line
-	9750 8500 9750 8750
-Wire Wire Line
-	8650 9200 8650 9550
-Wire Wire Line
-	9850 8500 9750 8500
-$Comp
-L Device:C_Small C4
-U 1 1 5E5E3F0A
-P 9950 8500
-F 0 "C4" V 9700 8650 50  0000 C CNN
-F 1 "10nF" V 9800 8650 50  0000 C CNN
-F 2 "Resistor_SMD:R_1206_3216Metric_Pad1.42x1.75mm_HandSolder" H 9950 8500 50  0001 C CNN
-F 3 "~" H 9950 8500 50  0001 C CNN
-	1    9950 8500
-	0    1    1    0
-$EndComp
-Wire Wire Line
-	10050 8500 10050 9550
-Wire Wire Line
-	10050 9550 8650 9550
-Connection ~ 8650 9550
-Wire Wire Line
-	8650 9550 8650 9650
 $Comp
 L Sensor_Temperature:TMP36xS U2
@@
 	7900 8350 7900 8150
 $Comp
-L trailTracer:Pad P2
-U 1 1 5E6A2F6F
-P 9900 8900
-F 0 "P2" V 9849 8828 50  0000 L CNN
-F 1 "Pad" V 9940 8828 50  0000 L CNN
-F 2 "trailTracer:Pad" H 9900 8950 50  0001 C CNN
-F 3 "" H 9900 8950 50  0001 C CNN
-	1    9900 8900
-	0    1    1    0
-$EndComp
-$Comp
-L trailTracer:Pad P3
-U 1 1 5E6A4BF6
-P 9900 9050
-F 0 "P3" V 9849 8978 50  0000 L CNN
-F 1 "Pad" V 9940 8978 50  0000 L CNN
-F 2 "trailTracer:Pad" H 9900 9100 50  0001 C CNN
-F 3 "" H 9900 9100 50  0001 C CNN
-	1    9900 9050
-	0    1    1    0
-$EndComp
-$Comp
-L trailTracer:Pad P6
-U 1 1 5E6F2C38
-P 9900 9200
-F 0 "P6" V 9849 9128 50  0000 L CNN
-F 1 "Pad" V 9940 9128 50  0000 L CNN
-F 2 "trailTracer:Pad" H 9900 9250 50  0001 C CNN
-F 3 "" H 9900 9250 50  0001 C CNN
-	1    9900 9200
-	0    1    1    0
-$EndComp
-$Comp
-L trailTracer:Pad P5
-U 1 1 5E6F7A3A
-P 8500 9050
-F 0 "P5" V 8449 8978 50  0000 L CNN
-F 1 "Pad" V 8540 8978 50  0000 L CNN
-F 2 "trailTracer:Pad" H 8500 9100 50  0001 C CNN
-F 3 "" H 8500 9100 50  0001 C CNN
-	1    8500 9050
-	0    -1   -1   0
-$EndComp
-$Comp
-L trailTracer:TE_OJ-SH-105LM U4
+L pihat-rescue:TE_OJ-SH-105LM-trailTracer U4
 U 1 1 5E6BDF85
 P 11650 9100
@@
 	0    1    1    0
 $EndComp
-$Comp
-L trailTracer:Pad P7
-U 1 1 5E6EBE98
-P 10750 8900
-F 0 "P7" H 10828 8738 50  0000 L CNN
-F 1 "Pad" H 10828 8647 50  0000 L CNN
-F 2 "trailTracer:Pad" H 10750 8950 50  0001 C CNN
-F 3 "" H 10750 8950 50  0001 C CNN
-	1    10750 8900
-	1    0    0    -1
-$EndComp
-Wire Wire Line
-	10750 9200 10750 9300
 Wire Wire Line
 	11050 9300 10750 9300
@@
 	1    0    0    -1
 $EndComp
-Text Notes 10250 8900 0    50   ~ 0
-P7: Jump to ATTiny85 output pad.\n
 $Comp
 L Device:R_Small R11
 U 1 1 5E71E70E
-P 8150 9150
-F 0 "R11" V 7954 9150 50  0000 C CNN
-F 1 "10K" V 8045 9150 50  0000 C CNN
-F 2 "Resistor_SMD:R_0805_2012Metric" H 8150 9150 50  0001 C CNN
-F 3 "~" H 8150 9150 50  0001 C CNN
-	1    8150 9150
+P 8150 9300
+F 0 "R11" V 7954 9300 50  0000 C CNN
+F 1 "10K" V 8045 9300 50  0000 C CNN
+F 2 "Resistor_SMD:R_0805_2012Metric" H 8150 9300 50  0001 C CNN
+F 3 "~" H 8150 9300 50  0001 C CNN
+	1    8150 9300
 	1    0    0    -1
 $EndComp
@@
 L power:GND #PWR01
 U 1 1 5E72F6C1
-P 8150 9350
-F 0 "#PWR01" H 8150 9100 50  0001 C CNN
-F 1 "GND" H 8155 9177 50  0000 C CNN
-F 2 "" H 8150 9350 50  0001 C CNN
-F 3 "" H 8150 9350 50  0001 C CNN
-	1    8150 9350
-	1    0    0    -1
-$EndComp
-Wire Wire Line
-	8150 9250 8150 9350
-$Comp
-L trailTracer:Pad P4
+P 8150 9500
+F 0 "#PWR01" H 8150 9250 50  0001 C CNN
+F 1 "GND" H 8155 9327 50  0000 C CNN
+F 2 "" H 8150 9500 50  0001 C CNN
+F 3 "" H 8150 9500 50  0001 C CNN
+	1    8150 9500
+	1    0    0    -1
+$EndComp
+Wire Wire Line
+	8150 9400 8150 9500
+$Comp
+L pihat-rescue:Pad-trailTracer P4
 U 1 1 5E6B9FE2
-P 7300 8900
-F 0 "P4" V 7300 8950 50  0000 R CNN
-F 1 "Pad" V 7400 9000 50  0000 R CNN
-F 2 "trailTracer:Pad" H 7300 8950 50  0001 C CNN
-F 3 "" H 7300 8950 50  0001 C CNN
-	1    7300 8900
+P 7300 9050
+F 0 "P4" V 7300 9100 50  0000 R CNN
+F 1 "Pad" V 7400 9150 50  0000 R CNN
+F 2 "trailTracer:Pad" H 7300 9100 50  0001 C CNN
+F 3 "" H 7300 9100 50  0001 C CNN
+	1    7300 9050
 	0    -1   -1   0
 $EndComp
@@
 L Device:R_Small R9
 U 1 1 5E641330
-P 7900 8900
-F 0 "R9" V 7704 8900 50  0000 C CNN
-F 1 "15K" V 7795 8900 50  0000 C CNN
-F 2 "Resistor_SMD:R_0805_2012Metric" H 7900 8900 50  0001 C CNN
-F 3 "~" H 7900 8900 50  0001 C CNN
-	1    7900 8900
+P 7900 9050
+F 0 "R9" V 7704 9050 50  0000 C CNN
+F 1 "15K" V 7795 9050 50  0000 C CNN
+F 2 "Resistor_SMD:R_0805_2012Metric" H 7900 9050 50  0001 C CNN
+F 3 "~" H 7900 9050 50  0001 C CNN
+	1    7900 9050
 	0    1    1    0
 $EndComp
 Wire Wire Line
-	8150 9050 8150 8900
-Wire Wire Line
-	8150 8900 8800 8900
-Wire Wire Line
-	8150 8900 8000 8900
-Connection ~ 8150 8900
-Wire Wire Line
-	7800 8900 7600 8900
+	8150 9200 8150 9050
+Wire Wire Line
+	8150 9050 8000 9050
+Wire Wire Line
+	7800 9050 7600 9050
 Text GLabel 12500 9650 2    50   Input ~ 0
 PI_5V
@@
 	13800 4650 13800 4900
 Connection ~ 13800 4650
+Text GLabel 8800 8900 0    50   Input ~ 0
+TINY_B4
+Text GLabel 10650 9100 0    50   Input ~ 0
+TINY_B4
+Wire Wire Line
+	10650 9100 10750 9100
+Wire Wire Line
+	10750 9100 10750 9300
+Wire Wire Line
+	8150 9050 8800 9050
+Connection ~ 8150 9050
+Wire Wire Line
+	9750 8750 9600 8750
+Text GLabel 9600 8900 2    50   Input ~ 0
+TINY_B2
+Text GLabel 8600 7750 2    50   Input ~ 0
+TINY_B2
+Wire Wire Line
+	5000 10000 5000 10100
+$Comp
+L power:GND #PWR0127
+U 1 1 5E9C521F
+P 5000 10100
+F 0 "#PWR0127" H 5000 9850 50  0001 C CNN
+F 1 "GND" H 5005 9927 50  0000 C CNN
+F 2 "" H 5000 10100 50  0001 C CNN
+F 3 "" H 5000 10100 50  0001 C CNN
+	1    5000 10100
+	1    0    0    -1
+$EndComp
+$Comp
+L Diode:B340 D5
+U 1 1 5E9C5225
+P 5000 9850
+F 0 "D5" V 5050 9950 50  0000 L CNN
+F 1 "B340" V 5150 9950 50  0000 L CNN
+F 2 "Diode_THT:D_DO-15_P5.08mm_Vertical_AnodeUp" H 5000 9675 50  0001 C CNN
+F 3 "http://www.jameco.com/Jameco/Products/ProdDS/1538777.pdf" H 5000 9850 50  0001 C CNN
+	1    5000 9850
+	0    1    1    0
+$EndComp
+Wire Wire Line
+	5000 9700 5000 9600
+Connection ~ 5000 9600
+Wire Wire Line
+	5000 9600 5100 9600
+Text GLabel 5550 1600 2    50   Input ~ 0
+GPIO_14
+Text GLabel 5550 1700 2    50   Input ~ 0
+GPIO_15
+Wire Wire Line
+	4650 9600 5000 9600
+Wire Wire Line
+	8650 9200 8650 9650
+Wire Wire Line
+	9750 8350 9750 8750
 $EndSCHEMATC
