File: KiCAD/PiHat/pihat/pihat.sch (KiCad schematic (older format))
At the start: 39 parts, among them J1 Pan Servo Connector, J2 Tilt Servo Connector, J3 Fan, J4 Power Connector, P1 Conn_02x20_Odd_Even, P4 Pad, Q1 BSS138, Q2 BSS138, U1 TPS5430-Q1, U2 TMP36xS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

Commit message: Added MOSFET switch, Logo, Prototype area
Parts:
- removed D2: 1N4001, Diode_THT:D_DO-41_SOD81_P10.16mm_Horizontal, symbol Diode:1N4001
- removed D4: LED, LED_THT:LED_D3.0mm, symbol Device:LED
- removed Q1, Q2: BSS138, Package_TO_SOT_SMD:SOT-23, symbol Transistor_FET:BSS138
- removed R12: 120R, Resistor_SMD:R_0805_2012Metric_Pad1.15x1.40mm_HandSolder, symbol Device:R_Small
- removed R5, R6: 220R, Resistor_SMD:R_0805_2012Metric, symbol Device:R_Small
- removed U2: TMP36xS, Package_SO:SOIC-8_3.9x4.9mm_P1.27mm, symbol Sensor_Temperature:TMP36xS
- removed U4: TE_OJ-SH-105LM, trailTracer:TE_OJ-SH-105LM, symbol pihat-rescue:TE_OJ-SH-105LM-trailTracer
- added C7: 100uF, Resistor_SMD:R_1206_3216Metric_Pad1.42x1.75mm_HandSolder, symbol Device:C
- added C8: 220pF, Resistor_SMD:R_1206_3216Metric_Pad1.42x1.75mm_HandSolder, symbol Device:C
- added C9: 10uF, Resistor_SMD:R_1206_3216Metric_Pad1.42x1.75mm_HandSolder, symbol Device:C
- added D1: LED, LED_THT:LED_D1.8mm_W3.3mm_H2.4mm, symbol Device:LED
- added Q1, Q2: 2N7000, Package_TO_SOT_THT:TO-92_Inline, symbol Transistor_FET:2N7000
- added R5: 220R, Resistor_SMD:R_1206_3216Metric_Pad1.42x1.75mm_HandSolder, symbol Device:R
- added U2: LMT87, Package_TO_SOT_THT:TO-92_Inline, symbol trailTracer:LMT87
- added U4: TPS22965, Package_SON:WSON-8-1EP_2x2mm_P0.5mm_EP0.9x1.6mm_ThermalVias, symbol trailTracer:TPS22965
- D5: footprint Diode_THT:D_DO-15_P5.08mm_Vertical_AnodeUp -> trailTracer:B340
- F1: value 5A Medium Blow -> Fuse; footprint Resistor_SMD:R_0603_1608Metric_Pad1.05x0.95mm_HandSolder -> trailTracer:Fuse_Holder_TR5
- U1: footprint Package_SO:SOIC-8-1EP_3.9x4.9mm_P1.27mm_EP2.41x3.81mm_ThermalVias -> trailTracer:SOIC-8-1EP_3.9x4.9mm_P1.27mm_EP2.29x3mm_ThermalVias
Connections:
- net GPIO_14 is gone; now on net TINY_B0: P1.8 (Pin_8)
- net GPIO_15 is gone; now on net TINY_B1: P1.10 (Pin_10)
- net +3V3: now also C7.2, Q1.2 (G), Q2.2 (G), U4.1 (Vin), U4.2 (Vin)
- net +5V: now also U2.1 (VCC), U4.4 (bias)
- net GND: now also C7.1, C8.2, C9.1, R5.2, U2.3 (GND), U4.5 (GND)
- net GPIO_2: now also R2.1, Q1.1 (S)
- net GPIO_3: now also R4.1, Q2.1 (S)
- net GPIO_4: no longer J3.2 (Pin_2)
- net PI_5V: now also C9.2, U4.7 (Vout), U4.8 (Vout)
- net TINY_B2: now also U2.2 (OUT)
- net TINY_B4: now also D1.2 (A), U4.3 (ON)
- net at J1.3 (Pin_3), R1.1: now also Q1.3 (D)
- net at J2.3 (Pin_3), R3.1: now also Q2.3 (D)
- net TINY_B0: now reaches U3.5 (PB0)
- net TINY_B1: now reaches U3.6 (PB1)
- new net: C8.1, U4.6 (CT)
- new net: D1.1 (K), R5.1
Other:
- moved on the sheet: C5
